Commit message: fix some errors for urdf

File: living_lab_robot_description/urdf/arm.urdf.xacro (robot description, xacro)
@@ -16,5 +16,5 @@
         <inertial>
             <origin xyz="0.0784 0 -0.0345" rpy="0 0 0"/>
-            <mass value="0.4997"/>
+            <mass value="0.04997"/>
             <inertia ixx="0.0007768" ixy="0.0" ixz="0.0" iyy="0.0023504" iyz="0.0" izz="0.0020179"/>
         </inertial>
@@ -44,5 +44,5 @@
         <inertial>
             <origin xyz="0.0330 0 0" rpy="0 0 0"/>
-            <mass value="0.5067"/>
+            <mass value="0.05067"/>
             <inertia ixx="0.0021992" ixy="0.0" ixz="0.0" iyy="0.0006670" iyz="0.0" izz="0.0021992"/>
         </inertial>
@@ -72,5 +72,5 @@
         <inertial>
             <origin xyz="0.1642 0 0.0083" rpy="0 0 0"/>
-            <mass value="0.9000"/>
+            <mass value="0.09000"/>
             <inertia ixx="0.0021659" ixy="0" ixz="0" iyy="0.0074914" iyz="0" izz="0.0086634"/>
         </inertial>
@@ -100,5 +100,5 @@
         <inertial>
             <origin xyz="0.1137 0 -0.0409" rpy="0 0 0"/>
-            <mass value="0.8000"/>
+            <mass value="0.08000"/>
             <inertia ixx="0.0013151" ixy="0" ixz="0" iyy="0.0034294" iyz="0.0" izz="0.0042325"/>
         </inertial>
@@ -128,5 +128,5 @@
         <inertial>
             <origin xyz="0.0269 0.0 0.0" rpy="0 0 0"/>
-            <mass value="0.2697"/>
+            <mass value="0.02697"/>
             <inertia ixx="00.0012527" ixy="0.0" ixz="0.0" iyy="0.0003956" iyz="0.0" izz="0.0012527"/>
         </inertial>
@@ -156,5 +156,5 @@
         <inertial>
             <origin xyz="0.0667 0 -0.0005" rpy="0 0 0"/>
-            <mass value="0.3885"/>
+            <mass value="0.03885"/>
             <inertia ixx="0.0005947" ixy="0.0" ixz="0.0" iyy="0.0005919" iyz="0.0" izz="0.0010050"/>
         </inertial>

File: living_lab_robot_description/urdf/body_assy.urdf.xacro (robot description, xacro)
@@ -16,5 +16,5 @@
         <inertial>
             <origin xyz="0 0 0.3780" rpy="0 0 0"/>
-            <mass value="3.21"/>
+            <mass value="30.21"/>
             <inertia ixx="0.263797" ixy="0.000014" ixz="-0.000365" iyy="0.255334" iyz="-0.000303" izz="0.069846"/>
         </inertial>
@@ -43,5 +43,5 @@
         <inertial>
             <origin xyz="0 0 0" rpy="0 0 0"/>
-            <mass value="0.31"/>
+            <mass value="10.31"/>
             <inertia ixx="0.001422" ixy="0" ixz="0" iyy="0.000917" iyz="0" izz="0.001769"/>
         </inertial>

File: living_lab_robot_description/urdf/head_assy.urdf.xacro (robot description, xacro)
@@ -17,5 +17,5 @@
         <inertial>
             <origin xyz="0 0 -0.1224" rpy="0 0 0"/>
-            <mass value="6.545411"/>
+            <mass value="16.545411"/>
             <inertia ixx="0.085366" ixy="0.0" ixz="0.0" iyy="0.085366" iyz="0.0" izz="0.105357"/>
         </inertial>
@@ -44,5 +44,5 @@
         <inertial>
             <origin xyz="0.014478 0.0 -0.045490" rpy="0 0 0"/>
-            <mass value="0.186690"/>
+            <mass value="10.186690"/>
             <inertia ixx="0.000811" ixy="0.0" ixz="0.000012" iyy="0.000271" iyz="0.0" izz="0.000576"/>
         </inertial>
@@ -71,5 +71,5 @@
         <inertial>
             <origin xyz="-0.098000 0 0.057616" rpy="0 0 0"/>
-            <mass value="2.540090"/>
+            <mass value="20.540090"/>
             <inertia ixx="0.022353" ixy="0.0" ixz="0.0" iyy="0.022353" iyz="0.0" izz="0.040886"/>
         </inertial>

Commit message: delete

File: living_lab_robot_description/urdf/arm.urdf.xacro (robot description, xacro)
@@ -197,3 +197,7 @@
     </joint>
     <xacro:insert_position_transmission name="arm6_joint" />
+    <xacro:sensor_d435 parent="head_tilt_unit">
+        <origin xyz="0.0172 0 0.0185" rpy="0 0 0"/>
+    </xacro:sensor_d435>
+    <xacro:insert_rgbd_camera_sensor name="camera"/>
 </robot>

Commit message: Fixed error

File: living_lab_robot_description/urdf/arm.urdf.xacro (robot description, xacro)
@@ -197,7 +197,3 @@
     </joint>
     <xacro:insert_position_transmission name="arm6_joint" />
-    <xacro:sensor_d435 parent="head_tilt_unit">
-        <origin xyz="0.0172 0 0.0185" rpy="0 0 0"/>
-    </xacro:sensor_d435>
-    <xacro:insert_rgbd_camera_sensor name="camera"/>
 </robot>
